File: KiCad/Epaper213.kicad_sch (KiCad schematic)
At the start: 34 parts, among them J1 USB-C, J2 DC, J3 Conn_01x02, M1 EPaper, U1 LMR16006+FB, U2 FT231XQ, U3 ESP32-PICO-MINI-02, U4 QR

Commit message: Both epaper boards
Parts:
- J3: footprint RevK:Molex_MiniSPOX_H2RA -> RevK:Molex_MiniSPOX_H3RA; symbol Connector_Generic:Conn_01x02 -> Connector_Generic:Conn_01x03
Connections:
- net BUTTON1: now reaches U3.24 (IO4)
- net BUTTON1: now also J3.2 (Pin_2)
- net BUTTON renamed BUTTON2
- net BUTTON2: now also J3.3 (Pin_3); no longer J3.2 (Pin_2)
- no-connect marks 14 -> 13
Other:
- title: 1.54" epaper display board -> 2.13" epaper display board
Changed lines of the file:
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@@
   (paper "A4")
   (title_block
-    (title "1.54\" epaper display board")
+    (title "2.13\" epaper display board")
     (date "${DATE}")
     (rev "1")
@@
   (no_connect (at 195.58 50.8))
   (no_connect (at 195.58 40.64))
-  (no_connect (at 195.58 63.5))
   (wire (pts (xy 55.88 33.02) (xy 58.42 33.02))
     (stroke (width 0) (type default) (color 0 0 0 0))
@@
     )
   )
+  (global_label "BUTTON2" (shape bidirectional) (at 198.12 104.14 180) (fields_autoplaced)
+    (effects (font (size 1.27 1.27)) (justify right))
+    (property "Intersheet References" "${INTERSHEET_REFS}" (id 0) (at 187.3896 104.0606 0)
+      (effects (font (size 1.27 1.27)) (justify right) hide)
+    )
+  )
   (global_label "BOOT" (shape input) (at 195.58 58.42 180) (fields_autoplaced)
     (effects (font (size 1.27 1.27)) (justify right))
@@
     )
   )
-  (global_label "BUTTON" (shape bidirectional) (at 198.12 104.14 180) (fields_autoplaced)
-    (effects (font (size 1.27 1.27)) (justify right))
-    (property "Intersheet References" "${INTERSHEET_REFS}" (id 0) (at 188.5991 104.0606 0)
+  (global_label "BUTTON1" (shape bidirectional) (at 198.12 101.6 180) (fields_autoplaced)
+    (effects (font (size 1.27 1.27)) (justify right))
+    (property "Intersheet References" "${INTERSHEET_REFS}" (id 0) (at 187.3896 101.5206 0)
       (effects (font (size 1.27 1.27)) (justify right) hide)
     )
@@
     )
   )
+  (global_label "BUTTON2" (shape bidirectional) (at 226.06 60.96 0) (fields_autoplaced)
+    (effects (font (size 1.27 1.27)) (justify left))
+    (property "Intersheet References" "${INTERSHEET_REFS}" (id 0) (at 236.7904 61.0394 0)
+      (effects (font (size 1.27 1.27)) (justify left) hide)
+    )
+  )
   (global_label "SRCS" (shape output) (at 226.06 78.74 0) (fields_autoplaced)
     (effects (font (size 1.27 1.27)) (justify left))
@@
     )
   )
-  (global_label "BUTTON" (shape bidirectional) (at 226.06 60.96 0) (fields_autoplaced)
-    (effects (font (size 1.27 1.27)) (justify left))
-    (property "Intersheet References" "${INTERSHEET_REFS}" (id 0) (at 235.5809 61.0394 0)
-      (effects (font (size 1.27 1.27)) (justify left) hide)
+  (global_label "BUTTON1" (shape bidirectional) (at 195.58 63.5 180) (fields_autoplaced)
+    (effects (font (size 1.27 1.27)) (justify right))
+    (property "Intersheet References" "${INTERSHEET_REFS}" (id 0) (at 184.8496 63.5794 0)
+      (effects (font (size 1.27 1.27)) (justify right) hide)
     )
   )
@@
     (pin "1")
   )
-  (symbol (lib_id "power:GND") (at 198.12 101.6 270) (unit 1)
+  (symbol (lib_id "power:GND") (at 198.12 99.06 270) (unit 1)
     (in_bom yes) (on_board yes) (fields_autoplaced)
-    (property "Reference" "#PWR019" (id 0) (at 191.77 101.6 0)
-      (effects (font (size 1.27 1.27)) hide)
-    )
-    (property "Value" "GND" (id 1) (at 194.9451 102.0338 90)
-      (effects (font (size 1.27 1.27)) (justify right))
-    )
-    (property "Footprint" "" (id 2) (at 198.12 101.6 0)
-      (effects (font (size 1.27 1.27)) hide)
-    )
-    (property "Datasheet" "" (id 3) (at 198.12 101.6 0)
+    (property "Reference" "#PWR019" (id 0) (at 191.77 99.06 0)
+      (effects (font (size 1.27 1.27)) hide)
+    )
+    (property "Value" "GND" (id 1) (at 194.9451 99.4938 90)
+      (effects (font (size 1.27 1.27)) (justify right))
+    )
+    (property "Footprint" "" (id 2) (at 198.12 99.06 0)
+      (effects (font (size 1.27 1.27)) hide)
+    )
+    (property "Datasheet" "" (id 3) (at 198.12 99.06 0)
       (effects (font (size 1.27 1.27)) hide)
     )
@@
     (pin "2")
   )
-  (symbol (lib_id "Connector_Generic:Conn_01x02") (at 203.2 101.6 0) (unit 1)
+  (symbol (lib_id "Connector_Generic:Conn_01x03") (at 203.2 101.6 0) (unit 1)
     (in_bom yes) (on_board yes) (fields_autoplaced)
     (property "Reference" "J3" (id 0) (at 205.232 102.0353 0)
@@
       (effects (font (size 1.27 1.27)) (justify left))
     )
-    (property "Footprint" "RevK:Molex_MiniSPOX_H2RA" (id 2) (at 203.2 101.6 0)
+    (property "Footprint" "RevK:Molex_MiniSPOX_H3RA" (id 2) (at 203.2 101.6 0)
       (effects (font (size 1.27 1.27)) hide)
     )
@@
     (pin "1")
     (pin "2")
+    (pin "3")
   )
   (symbol (lib_id "power:+3.3V") (at 226.06 38.1 270) (unit 1)
@@
     )
     (path "/ca6f103f-48cc-446d-9d86-158c35366e6f"
-      (reference "J3") (unit 1) (value "Conn_01x02") (footprint "RevK:Molex_MiniSPOX_H2RA")
+      (reference "J3") (unit 1) (value "Conn_01x02") (footprint "RevK:Molex_MiniSPOX_H3RA")
     )
     (path "/00000000-0000-0000-0000-0000610fe01a"
