File: KiCad/Epaper154.kicad_pcb (KiCad board)
At the start: 2 copper layers, 58.2 x 37 mm, 32 parts, among them J1 USB-C, J2 DC, J3 TEMP, M1 OLED1.5-RGB, U1 LMR16006+FB, U2 SCD41, U3 FT231XQ, U4 ESP32-PICO-MINI-02, U5 QR

Commit message: Starting new PCB
Parts:
- removed M1: OLED1.5-RGB, RevK:OLED1.5-RGB
- removed the U2 at (91.8, 68.5)
- renumbered R13 to R10, R7 to R11, R8 to R12, R9 to R13, R10 to R7, R11 to R8, R12 to R9, U3 to U2, U4 to U3, U5 to U4
Connections:
- U3 pad 12: OLED-MOSI -> unconnected-(U3-Pad12)
- U3 pad 13: OLED-SCLK -> unconnected-(U3-Pad13)
- U3 pad 15: OLED-CS0 -> unconnected-(U3-Pad15)
- U3 pad 16: OLED-DC -> unconnected-(U3-Pad16)
- U3 pad 17: OLED-RST -> unconnected-(U3-Pad17)
- U3 pad 34: CO2-SDA -> unconnected-(U3-Pad34)
- U3 pad 35: CO2-SCL -> unconnected-(U3-Pad35)
Routing:
- net unconnected-(U3-Pad35): track 0.00 -> 52.1 mm, vias 0 -> 2
- net CO2-SCL: track 52.1 -> 0.00 mm, vias 2 -> 0
- net unconnected-(U3-Pad34): track 0.00 -> 48.4 mm, vias 0 -> 4
- net CO2-SDA: track 48.4 -> 0.00 mm, vias 4 -> 0
- net unconnected-(U3-Pad17): track 0.00 -> 22.6 mm
- net OLED-RST: track 22.6 -> 0.00 mm
- net unconnected-(U3-Pad16): track 0.00 -> 21.1 mm
- net OLED-DC: track 21.1 -> 0.00 mm
- net unconnected-(U3-Pad15): track 0.00 -> 19.6 mm
- net OLED-CS0: track 19.6 -> 0.00 mm
- net unconnected-(U3-Pad13): track 0.00 -> 17.2 mm
- net OLED-SCLK: track 17.2 -> 0.00 mm
- net unconnected-(U3-Pad12): track 0.00 -> 15.9 mm
- net OLED-MOSI: track 15.9 -> 0.00 mm

Commit message: Started
Parts:
- removed J3: TEMP, RevK:Molex_MiniSPOX_H3RA
- removed R10: 4k7, RevK:R_0603
- added M1: EPaper, Connector_PinHeader_2.54mm:PinHeader_1x13_P2.54mm_Vertical, F.Cu at (135.9, 101.6)
- D2: footprint Diode_SMD:D_1206_3216Metric -> RevK:D_1206
- U4: footprint RevK:QR-ENVMON -> RevK:QR-GFX; moved to F.Cu
- moved J1 47.4 mm to (166.4, 82.5), turned to 90 degrees
- moved U4 42.8 mm to (151.0, 65.3)
- moved C4 39.8 mm to (160.0, 64.8), turned to 0 degrees
- moved R5 35.9 mm to (156.2, 76.2), turned to 0 degrees
- moved R3 35.6 mm to (152.4, 77.5), turned to 0 degrees
- moved Logo2 33.3 mm to (141.0, 64.8)
- moved U2 33.0 mm to (154.9, 82.5)
- moved R9 31.1 mm to (146.1, 71.1), turned to 0 degrees
- moved R13 30.5 mm to (151.1, 94.4), turned to 0 degrees
- moved R11 29.9 mm to (147.7, 96.5), turned to 0 degrees
- moved U1 29.6 mm to (158.3, 68.8), turned to 0 degrees
- moved R7 27.8 mm to (151.1, 74.9), turned to 0 degrees
- moved R8 26.5 mm to (151.1, 96.5), turned to 0 degrees
- moved R6 25.7 mm to (142.4, 74.2), turned to 0 degrees
- moved R2 24.9 mm to (151.1, 72.8)
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Routing:
- net +3V3: track 128.4 -> 0.00 mm, vias 3 -> 0
- net unconnected-(U3-Pad35): track 52.1 -> 0.00 mm, vias 2 -> 0
- net GND: track 50.1 -> 0.00 mm, vias 5 -> 0
- net unconnected-(U3-Pad34): track 48.4 -> 0.00 mm, vias 4 -> 0
- net O: track 25.3 -> 0.00 mm, vias 2 -> 0
- net unconnected-(U3-Pad17): track 22.6 -> 0.00 mm
- net TEMP: track 21.8 -> 0.00 mm
- net unconnected-(U3-Pad16): track 21.1 -> 0.00 mm
- net unconnected-(U3-Pad15): track 19.6 -> 0.00 mm
- net DC: track 19.1 -> 0.00 mm
- net VBUS: track 18.3 -> 0.00 mm, vias 2 -> 0
- net EN: track 17.5 -> 0.00 mm, vias 2 -> 0
- net unconnected-(U3-Pad13): track 17.2 -> 0.00 mm
- net unconnected-(U3-Pad12): track 15.9 -> 0.00 mm
- net I: track 14.8 -> 0.00 mm, vias 2 -> 0
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Other:
- board size 58.2 x 37 mm -> 43.2 x 43.2 mm
- board text removed: "14"
- board text removed: "25"
- board text removed: "26"
- board text removed: "27"
- board text removed: "3.3"
- board text removed: "32"
- board text removed: "33"
- board text removed: "CO₂"
- board text removed: "DC 4V-60V"
- board text removed: "DS18B20"
- board text removed: "Environmental Monitor"
- board text removed: "LED: 7/19/8"
- board text removed: "SCD41 SCL: 21 SDA: 22"
- board text removed: "⏚"

Commit message: Epaper PCB
Parts:
- added H1: MountingHole, RevK:Hole-2.5mm, F.Cu at (170.2, 63.5)
- added H2: MountingHole, RevK:Hole-2.5mm, F.Cu at (132.1, 63.5)
- added H3: MountingHole, RevK:Hole-2.5mm, F.Cu at (132.1, 101.6)
- added H4: MountingHole, RevK:Hole-2.5mm, F.Cu at (170.2, 101.6)
- added J3: Conn_01x02, RevK:Molex_MiniSPOX_H2RA, F.Cu at (159.4, 71.8)
- Logo1: moved to F.Cu
- Logo2, U4: moved to B.Cu
- moved R10 33.2 mm to (141.0, 64.0), turned to -90 degrees
- moved R12 31.7 mm to (142.2, 64.0), turned to -90 degrees
- moved R8 25.6 mm to (155.2, 71.3)
- moved Logo1 21.2 mm to (160.9, 63.7), turned to 90 degrees
- moved U4 21.1 mm to (163.2, 82.5), turned to 90 degrees
- moved R9 20.5 mm to (138.4, 90.2)
- moved Logo2 19.9 mm to (160.9, 64.9), turned to -90 degrees
- moved R4 17.8 mm to (158.1, 80.0), turned to 90 degrees
- moved D2 14.3 mm to (156.8, 90.8), turned to 90 degrees
- moved R6 13.2 mm to (153.7, 81.3), turned to 90 degrees
- moved R2 10.3 mm to (145.0, 64.5)
- moved U1 9.67 mm to (149.4, 65.0)
- moved R3 9.53 mm to (158.1, 85.1), turned to -90 degrees
- moved R1 9.23 mm to (145.0, 63.2), turned to 180 degrees
- moved R11 8.08 mm to (139.7, 64.0), turned to -90 degrees
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- renumbered R11 to R10, R12 to R11, R13 to R12
Connections:
- M1 pad 10: unconnected-(M1-Pad10) -> SDCS
- M1 pad 11: unconnected-(M1-Pad11) -> RST
- M1 pad 12: unconnected-(M1-Pad12) -> BUSY
- M1 pad 13: unconnected-(M1-Pad13) -> ENA
- M1 pad 2: unconnected-(M1-Pad2) -> +3V3
- M1 pad 3: unconnected-(M1-Pad3) -> GND
- M1 pad 4: unconnected-(M1-Pad4) -> SCK
- M1 pad 5: unconnected-(M1-Pad5) -> MISO
- M1 pad 6: unconnected-(M1-Pad6) -> MOSI
- M1 pad 7: unconnected-(M1-Pad7) -> CS
- M1 pad 8: unconnected-(M1-Pad8) -> D/C
- M1 pad 9: unconnected-(M1-Pad9) -> SRCS
- U3 pad 12: unconnected-(U3-Pad12) -> MISO
- U3 pad 13: unconnected-(U3-Pad13) -> SRCS
- U3 pad 15: unconnected-(U3-Pad15) -> SDCS
- U3 pad 16: unconnected-(U3-Pad16) -> RST
- U3 pad 17: unconnected-(U3-Pad17) -> BUSY
- U3 pad 18: TEMP -> SCK
- U3 pad 20: unconnected-(U3-Pad20) -> ENA
- U3 pad 26: unconnected-(U3-Pad26) -> BUTTON
- U3 pad 29: unconnected-(U3-Pad29) -> CS
- U3 pad 34: unconnected-(U3-Pad34) -> MOSI
- U3 pad 35: unconnected-(U3-Pad35) -> D/C
Routing:
- net +3V3: track 0.00 -> 90.0 mm, vias 0 -> 4
- net DC: track 0.00 -> 45.8 mm, vias 0 -> 1
- net ENA: track 0.00 -> 35.9 mm
- net D/C: track 0.00 -> 35.7 mm, vias 0 -> 1
- net GND: track 0.00 -> 32.1 mm, vias 0 -> 3
- net BUSY: track 0.00 -> 30.9 mm
- net MOSI: track 0.00 -> 28.5 mm, vias 0 -> 1
- net CS: track 0.00 -> 28.4 mm, vias 0 -> 1
- net RST: track 0.00 -> 27.8 mm
- net EN: track 0.00 -> 27.3 mm, vias 0 -> 2
- net SCK: track 0.00 -> 25.6 mm, vias 0 -> 1
- net SDCS: track 0.00 -> 24.8 mm
- net VBUS: track 0.00 -> 23.4 mm, vias 0 -> 2
- net SRCS: track 0.00 -> 21.2 mm
- net BUTTON: track 0.00 -> 18.8 mm, vias 0 -> 1
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Other:
- board text added: "13"
- board text added: "14"
- board text added: "20"
- board text added: "21"
- board text added: "22"
- board text added: "25"
- board text added: "26"
- board text added: "27"
- board text added: "32"
- board text added: "33"
- board text added: "5"
- board text added: "DC 4V-60V"
- board text added: "Epaper Display Board"
- board text added: "RGB: 7/19/8"

Commit message: Both epaper boards
Parts:
- J3: footprint RevK:Molex_MiniSPOX_H2RA -> RevK:Molex_MiniSPOX_H3RA
- moved Logo1 36.7 mm to (141.5, 94.7)
- moved C1 27.5 mm to (147.3, 65.3), turned to 90 degrees
- moved D1 26.0 mm to (151.7, 68.2)
- moved C3 25.3 mm to (154.8, 68.6), turned to 90 degrees
- moved Logo2 24.5 mm to (149.1, 86.4)
- moved C2 24.5 mm to (148.6, 68.6), turned to 90 degrees
- moved L1 14.4 mm to (153.3, 65.0)
- moved J3 0.13 mm to (159.4, 71.6)
Connections:
- J3 pad 2: BUTTON -> BUTTON1
- U3 pad 24: unconnected-(U3-Pad24) -> BUTTON1
- U3 pad 26: BUTTON -> BUTTON2
Routing:
- net BUTTON1: track 0.00 -> 21.0 mm, vias 0 -> 1
- net BUTTON2: track 0.00 -> 19.5 mm, vias 0 -> 1
- net BUTTON: track 18.8 -> 0.00 mm, vias 1 -> 0
- net DC: track 45.8 -> 48.0 mm
- net I: track 16.0 -> 17.2 mm
- net BOOT: track 11.3 -> 12.3 mm
- net GND: track 32.1 -> 31.3 mm
Other:
- outline, holes or cut-outs redrawn
- board text added: "4"
- board text added: "⏚"

Commit message: Tidy
Routing:
- net ENA: track 35.9 -> 37.0 mm
- net BUSY: track 30.9 -> 32.0 mm
- net RST: track 27.8 -> 28.9 mm
- net SRCS: track 21.2 -> 22.2 mm
- net SDCS: track 24.8 -> 25.8 mm
- net GND: vias 3 -> 4
Changed lines of the file:
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@@
   (via (at 151.892 71.12) (size 0.8) (drill 0.4) (layers "F.Cu" "B.Cu") (free) (net 11))
   (via (at 151.892 68.072) (size 0.8) (drill 0.4) (layers "F.Cu" "B.Cu") (net 11))
+  (via (at 148.082 82.55) (size 0.8) (drill 0.4) (layers "F.Cu" "B.Cu") (free) (net 11))
   (arc (start 152.03 68.21) (mid 151.932419 68.169581) (end 151.892 68.072) (width 0.5) (layer "F.Cu") (net 11))
   (arc (start 152.67 87.99) (mid 154.60456 92.66044) (end 159.275 94.595) (width 0.25) (layer "F.Cu") (net 11))
@@
   (segment (start 138.295 63.133) (end 139.65 63.133) (width 0.25) (layer "F.Cu") (net 30))
   (arc (start 139.65 63.133) (mid 139.685355 63.147645) (end 139.7 63.183) (width 0.25) (layer "F.Cu") (net 30))
-  (segment (start 147.828 87.20475) (end 147.828 94.742) (width 0.25) (layer "F.Cu") (net 34))
-  (segment (start 151.638 98.552) (end 153.162 98.552) (width 0.25) (layer "F.Cu") (net 34))
+  (segment (start 151.384 100.33) (end 154.94 100.33) (width 0.25) (layer "F.Cu") (net 34))
   (segment (start 146.52325 86.55) (end 147.17325 86.55) (width 0.25) (layer "F.Cu") (net 34))
-  (arc (start 147.828 94.742) (mid 148.943923 97.436077) (end 151.638 98.552) (width 0.25) (layer "F.Cu") (net 34))
-  (arc (start 153.162 98.552) (mid 155.317261 99.444739) (end 156.21 101.6) (width 0.25) (layer "F.Cu") (net 34))
+  (segment (start 147.828 87.20475) (end 147.828 96.774) (width 0.25) (layer "F.Cu") (net 34))
+  (arc (start 154.94 100.33) (mid 155.838026 100.701974) (end 156.21 101.6) (width 0.25) (layer "F.Cu") (net 34))
   (arc (start 147.17325 86.55) (mid 147.636228 86.741772) (end 147.828 87.20475) (width 0.25) (layer "F.Cu") (net 34))
+  (arc (start 147.828 96.774) (mid 148.869528 99.288472) (end 151.384 100.33) (width 0.25) (layer "F.Cu") (net 34))
   (segment (start 151.77 75.835) (end 150.511 75.835) (width 0.25) (layer "F.Cu") (net 35))
   (segment (start 140.82325 78.12475) (end 140.82325 76.65) (width 0.25) (layer "F.Cu") (net 35))
@@
   (arc (start 150.114 75.438) (mid 149.96521 75.79721) (end 149.606 75.946) (width 0.25) (layer "B.Cu") (net 35))
   (arc (start 143.002 75.946) (mid 141.385554 76.615554) (end 140.716 78.232) (width 0.25) (layer "B.Cu") (net 35))
-  (segment (start 151.638 98.044) (end 155.194 98.044) (width 0.25) (layer "F.Cu") (net 36))
-  (segment (start 148.336 86.76275) (end 148.336 94.742) (width 0.25) (layer "F.Cu") (net 36))
+  (segment (start 148.336 86.76275) (end 148.336 96.774) (width 0.25) (layer "F.Cu") (net 36))
+  (segment (start 151.384 99.822) (end 156.972 99.822) (width 0.25) (layer "F.Cu") (net 36))
   (arc (start 146.52325 84.95) (mid 147.805058 85.480942) (end 148.336 86.76275) (width 0.25) (layer "F.Cu") (net 36))
-  (arc (start 148.336 94.742) (mid 149.303133 97.076867) (end 151.638 98.044) (width 0.25) (layer "F.Cu") (net 36))
-  (arc (start 155.194 98.044) (mid 157.708472 99.085528) (end 158.75 101.6) (width 0.25) (layer "F.Cu") (net 36))
-  (segment (start 151.892 97.536) (end 157.226 97.536) (width 0.25) (layer "F.Cu") (net 38))
-  (segment (start 148.844 86.47075) (end 148.844 94.488) (width 0.25) (layer "F.Cu") (net 38))
-  (arc (start 148.844 94.488) (mid 149.736739 96.643261) (end 151.892 97.536) (width 0.25) (layer "F.Cu") (net 38))
+  (arc (start 148.336 96.774) (mid 149.228739 98.929261) (end 151.384 99.822) (width 0.25) (layer "F.Cu") (net 36))
+  (arc (start 156.972 99.822) (mid 158.229236 100.342764) (end 158.75 101.6) (width 0.25) (layer "F.Cu") (net 36))
+  (segment (start 151.384 99.314) (end 159.004 99.314) (width 0.25) (layer "F.Cu") (net 38))
+  (segment (start 148.844 86.47075) (end 148.844 96.774) (width 0.25) (layer "F.Cu") (net 38))
   (arc (start 146.52325 84.15) (mid 148.164268 84.829732) (end 148.844 86.47075) (width 0.25) (layer "F.Cu") (net 38))
-  (arc (start 157.226 97.536) (mid 160.099682 98.726318) (end 161.29 101.6) (width 0.25) (layer "F.Cu") (net 38))
+  (arc (start 159.004 99.314) (mid 160.620446 99.983554) (end 161.29 101.6) (width 0.25) (layer "F.Cu") (net 38))
+  (arc (start 148.844 96.774) (mid 149.587949 98.570051) (end 151.384 99.314) (width 0.25) (layer "F.Cu") (net 38))
   (segment (start 142.24 72.898) (end 152.325002 72.898) (width 0.25) (layer "F.Cu") (net 39))
   (segment (start 154.17 74.742998) (end 154.17 74.935) (width 0.25) (layer "F.Cu") (net 39))
@@
   (arc (start 141.62325 73.51475) (mid 141.803892 73.078642) (end 142.24 72.898) (width 0.25) (layer "F.Cu") (net 39))
   (arc (start 152.325002 72.898) (mid 153.629613 73.438387) (end 154.17 74.742998) (width 0.25) (layer "F.Cu") (net 39))
+  (segment (start 140.017 89.408) (end 142.26525 89.408) (width 0.25) (layer "F.Cu") (net 40))
   (segment (start 143.22325 87.8) (end 143.22325 88.45) (width 0.25) (layer "F.Cu") (net 40))
   (segment (start 144.272 87.376) (end 143.64725 87.376) (width 0.25) (layer "F.Cu") (net 40))
-  (segment (start 151.345643 74.168857) (end 150.876 74.6385) (width 0.25) (layer "F.Cu") (net 40))
-  (segment (start 143.22325 89.1) (end 143.22325 88.45) (width 0.25) (layer "F.Cu") (net 40))
   (segment (start 152.848883 74.168857) (end 151.345643 74.168857) (width 0.25) (layer "F.Cu") (net 40))
   (segment (start 153.17 74.935) (end 153.17 74.537672) (width 0.25) (layer "F.Cu") (net 40))
-  (segment (start 139.255 90.17) (end 142.15325 90.17) (width 0.25) (layer "F.Cu") (net 40))
   (via (at 150.876 74.6385) (size 0.8) (drill 0.4) (layers "F.Cu" "B.Cu") (net 40))
   (via (at 144.272 87.376) (size 0.8) (drill 0.4) (layers "F.Cu" "B.Cu") (net 40))
   (arc (start 143.64725 87.376) (mid 143.347437 87.500187) (end 143.22325 87.8) (width 0.25) (layer "F.Cu") (net 40))
   (arc (start 153.17 74.537672) (mid 153.078262 74.29393) (end 152.848883 74.168857) (width 0.25) (layer "F.Cu") (net 40))
-  (arc (start 142.15325 90.17) (mid 142.909854 89.856604) (end 143.22325 89.1) (width 0.25) (layer "F.Cu") (net 40))
+  (arc (start 151.345643 74.168857) (mid 151.013555 74.306412) (end 150.876 74.6385) (width 0.25) (layer "F.Cu") (net 40))
+  (arc (start 142.26525 89.408) (mid 142.942658 89.127408) (end 143.22325 88.45) (width 0.25) (layer "F.Cu") (net 40))
+  (arc (start 139.255 90.17) (mid 139.478185 89.631185) (end 140.017 89.408) (width 0.25) (layer "F.Cu") (net 40))
   (segment (start 150.873997 74.640503) (end 150.876 74.6385) (width 0.25) (layer "B.Cu") (net 40))
   (segment (start 150.873997 75.777631) (end 150.873997 74.640503) (width 0.25) (layer "B.Cu") (net 40))
@@
   (arc (start 155.770675 82.105) (mid 156.352095 82.220652) (end 156.845 82.55) (width 0.25) (layer "F.Cu") (net 45))
   (arc (start 160.45 82.8) (mid 160.303553 83.153553) (end 159.95 83.3) (width 0.25) (layer "F.Cu") (net 45))
-  (segment (start 151.892 97.028) (end 159.258 97.028) (width 0.25) (layer "F.Cu") (net 46))
-  (segment (start 149.352 86.17875) (end 149.352 94.488) (width 0.25) (layer "F.Cu") (net 46))
+  (segment (start 151.384 98.806) (end 161.036 98.806) (width 0.25) (layer "F.Cu") (net 46))
+  (segment (start 149.352 86.17875) (end 149.352 96.774) (width 0.25) (layer "F.Cu") (net 46))
+  (arc (start 149.352 96.774) (mid 149.947159 98.210841) (end 151.384 98.806) (width 0.25) (layer "F.Cu") (net 46))
+  (arc (start 161.036 98.806) (mid 163.011656 99.624344) (end 163.83 101.6) (width 0.25) (layer "F.Cu") (net 46))
   (arc (start 146.52325 83.35) (mid 148.523478 84.178522) (end 149.352 86.17875) (width 0.25) (layer "F.Cu") (net 46))
-  (arc (start 159.258 97.028) (mid 162.490892 98.367108) (end 163.83 101.6) (width 0.25) (layer "F.Cu") (net 46))
-  (arc (start 149.352 94.488) (mid 150.095949 96.284051) (end 151.892 97.028) (width 0.25) (layer "F.Cu") (net 46))
-  (segment (start 151.892 96.52) (end 161.29 96.52) (width 0.25) (layer "F.Cu") (net 47))
-  (segment (start 149.86 83.63675) (end 149.86 94.488) (width 0.25) (layer "F.Cu") (net 47))
+  (segment (start 149.86 83.63675) (end 149.86 96.774) (width 0.25) (layer "F.Cu") (net 47))
   (segment (start 146.52325 80.95) (end 147.17325 80.95) (width 0.25) (layer "F.Cu") (net 47))
-  (arc (start 161.29 96.52) (mid 164.882102 98.007898) (end 166.37 101.6) (width 0.25) (layer "F.Cu") (net 47))
+  (segment (start 151.384 98.298) (end 163.068 98.298) (width 0.25) (layer "F.Cu") (net 47))
+  (arc (start 149.86 96.774) (mid 150.306369 97.851631) (end 151.384 98.298) (width 0.25) (layer "F.Cu") (net 47))
   (arc (start 147.17325 80.95) (mid 149.073069 81.736931) (end 149.86 83.63675) (width 0.25) (layer "F.Cu") (net 47))
-  (arc (start 149.86 94.488) (mid 150.455159 95.924841) (end 151.892 96.52) (width 0.25) (layer "F.Cu") (net 47))
+  (arc (start 163.068 98.298) (mid 165.402867 99.265133) (end 166.37 101.6) (width 0.25) (layer "F.Cu") (net 47))
   (segment (start 146.52325 77.75) (end 146.72325 77.75) (width 0.25) (layer "F.Cu") (net 49))
   (segment (start 147.574 76.89925) (end 147.574 74.93) (width 0.25) (layer "F.Cu") (net 49))

Commit message: Shelly as well for low power
Parts:
- added J2: Shelly, RevK:Shelly, B.Cu at (154.0, 90.1)
- moved Logo2 4.33 mm to (148.2, 90.6)
- renumbered J2 to J3, J3 to J4
Routing:
- net I: track 17.2 -> 47.0 mm, vias 0 -> 1
- net O: track 14.4 -> 34.9 mm
- net BOOT: track 12.3 -> 26.6 mm
- net +3V3: track 90.3 -> 104.1 mm
- net GND: track 31.3 -> 20.1 mm, vias 4 -> 6
- net VBUS: track 23.4 -> 24.1 mm
