File: KiCad/Epaper154.kicad_sch (KiCad schematic)
At the start: 32 parts, among them J1 USB-C, J2 DC, J3 TEMP, M1 OLED1.5-RGB, U1 LMR16006+FB, U2 SCD41, U3 FT231XQ, U4 ESP32-PICO-MINI-02, U5 QR

Commit message: Starting new PCB
Parts:
- removed M1: OLED1.5-RGB, RevK:OLED1.5-RGB, symbol RevK:OLED1.5-RGB
- removed U2: SCD41, RevK:SCD41, symbol RevK:SCD41
- added M1: EPaper, symbol RevK:EPaper
- renumbered R13 to R10, R7 to R11, R8 to R12, R9 to R13, R10 to R7, R11 to R8, R12 to R9, U3 to U2, U4 to U3, U5 to U4
Connections:
- net CO2-SCL: no longer names the net of U3.35 (IO21)
- net CO2-SDA: no longer names the net of U3.34 (IO22)
- net OLED-CS0: no longer names the net of U3.15 (IO25)
- net OLED-DC: no longer names the net of U3.16 (IO26)
- net OLED-MOSI: no longer names the net of U3.12 (IO32)
- net OLED-RST: no longer names the net of U3.17 (IO27)
- net OLED-SCLK: no longer names the net of U3.13 (IO33)
Other:
- title: 1.5" OLED Module driver with GPIO -> 1.54" epaper display board
- moved on the sheet: D3, R11, R12, R13

Commit message: Started
Parts:
- removed J3: TEMP, RevK:Molex_MiniSPOX_H3RA, symbol Connector_Generic:Conn_01x03
- removed R10: 4k7, RevK:R_0603, symbol Device:R
- D2: footprint Diode_SMD:D_1206_3216Metric -> RevK:D_1206
- M1: footprint (none) -> Connector_PinHeader_2.54mm:PinHeader_1x13_P2.54mm_Vertical
- U4: footprint RevK:QR-ENVMON -> RevK:QR-GFX
Changed lines of the file:
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@@
-    )
-  )
-  (global_label "TEMP" (shape bidirectional) (at 198.12 134.62 180) (fields_autoplaced)
-    (effects (font (size 1.27 1.27)) (justify right))
-    (property "Intersheet References" "${INTERSHEET_REFS}" (id 0) (at 190.9577 134.6994 0)
-      (effects (font (size 1.27 1.27)) (justify right) hide)
     )
   )
@@
     (property "Intersheet References" "${INTERSHEET_REFS}" (id 0) (at 114.3 -36.195 0)
       (effects (font (size 1.27 1.27)) hide)
-    )
-  )
-  (global_label "TEMP" (shape bidirectional) (at 193.04 124.46 180) (fields_autoplaced)
-    (effects (font (size 1.27 1.27)) (justify right))
-    (property "Intersheet References" "${INTERSHEET_REFS}" (id 0) (at 185.8777 124.3806 0)
-      (effects (font (size 1.27 1.27)) (justify right) hide)
     )
   )
@@
     (pin "1")
   )
-  (symbol (lib_id "power:GND") (at 198.12 132.08 270) (unit 1)
-    (in_bom yes) (on_board yes) (fields_autoplaced)
-    (property "Reference" "#PWR017" (id 0) (at 191.77 132.08 0)
-      (effects (font (size 1.27 1.27)) hide)
-    )
-    (property "Value" "GND" (id 1) (at 194.9451 132.5138 90)
-      (effects (font (size 1.27 1.27)) (justify right))
-    )
-    (property "Footprint" "" (id 2) (at 198.12 132.08 0)
-      (effects (font (size 1.27 1.27)) hide)
-    )
-    (property "Datasheet" "" (id 3) (at 198.12 132.08 0)
-      (effects (font (size 1.27 1.27)) hide)
-    )
-    (pin "1")
-  )
   (symbol (lib_id "power:VBUS") (at 74.295 27.94 0) (unit 1)
     (in_bom yes) (on_board yes)
@@
     )
     (pin "1")
-  )
-  (symbol (lib_id "Connector_Generic:Conn_01x03") (at 203.2 134.62 0) (unit 1)
-    (in_bom no) (on_board yes) (fields_autoplaced)
-    (property "Reference" "J3" (id 0) (at 205.232 133.7853 0)
-      (effects (font (size 1.27 1.27)) (justify left))
-    )
-    (property "Value" "TEMP" (id 1) (at 205.232 136.3222 0)
-      (effects (font (size 1.27 1.27)) (justify left))
-    )
-    (property "Footprint" "RevK:Molex_MiniSPOX_H3RA" (id 2) (at 203.2 134.62 0)
-      (effects (font (size 1.27 1.27)) hide)
-    )
-    (property "Datasheet" "~" (id 3) (at 203.2 134.62 0)
-      (effects (font (size 1.27 1.27)) hide)
-    )
-    (pin "1")
-    (pin "2")
-    (pin "3")
   )
   (symbol (lib_id "power:GND") (at 86.995 33.02 90) (unit 1)
@@
     (pin "1")
   )
-  (symbol (lib_id "Device:R") (at 196.85 124.46 90) (unit 1)
-    (in_bom yes) (on_board yes)
-    (property "Reference" "R10" (id 0) (at 198.12 121.92 90)
-      (effects (font (size 1.27 1.27)) (justify left))
-    )
-    (property "Value" "4k7" (id 1) (at 198.755 124.46 90)
-      (effects (font (size 1.27 1.27)) (justify left))
-    )
-    (property "Footprint" "RevK:R_0603" (id 2) (at 196.85 126.238 90)
-      (effects (font (size 1.27 1.27)) hide)
-    )
-    (property "Datasheet" "~" (id 3) (at 196.85 124.46 0)
-      (effects (font (size 1.27 1.27)) hide)
-    )
-    (pin "1")
-    (pin "2")
-  )
-  (symbol (lib_id "power:+3.3V") (at 198.12 137.16 90) (unit 1)
-    (in_bom yes) (on_board yes) (fields_autoplaced)
-    (property "Reference" "#PWR018" (id 0) (at 201.93 137.16 0)
-      (effects (font (size 1.27 1.27)) hide)
-    )
-    (property "Value" "+3.3V" (id 1) (at 194.945 137.5938 90)
-      (effects (font (size 1.27 1.27)) (justify left))
-    )
-    (property "Footprint" "" (id 2) (at 198.12 137.16 0)
-      (effects (font (size 1.27 1.27)) hide)
-    )
-    (property "Datasheet" "" (id 3) (at 198.12 137.16 0)
-      (effects (font (size 1.27 1.27)) hide)
-    )
-    (pin "1")
-  )
   (symbol (lib_id "RevK:QR") (at 271.78 172.72 0) (unit 1)
     (in_bom no) (on_board yes) (fields_autoplaced)
@@
       (effects (font (size 1.27 1.27)) hide)
     )
-    (property "Footprint" "RevK:QR-ENVMON" (id 2) (at 271.145 173.355 0)
+    (property "Footprint" "RevK:QR-GFX" (id 2) (at 271.145 173.355 0)
       (effects (font (size 1.27 1.27)) hide)
     )
@@
       (effects (font (size 1.27 1.27)) (justify left))
     )
-    (property "Footprint" "" (id 2) (at 135.89 91.44 0)
+    (property "Footprint" "Connector_PinHeader_2.54mm:PinHeader_1x13_P2.54mm_Vertical" (id 2) (at 135.89 91.44 0)
       (effects (font (size 1.27 1.27)) hide)
     )
@@
     (pin "1")
     (pin "2")
-  )
-  (symbol (lib_id "power:+3.3V") (at 200.66 124.46 270) (unit 1)
-    (in_bom yes) (on_board yes) (fields_autoplaced)
-    (property "Reference" "#PWR019" (id 0) (at 196.85 124.46 0)
-      (effects (font (size 1.27 1.27)) hide)
-    )
-    (property "Value" "+3.3V" (id 1) (at 203.835 124.8938 90)
-      (effects (font (size 1.27 1.27)) (justify left))
-    )
-    (property "Footprint" "" (id 2) (at 200.66 124.46 0)
-      (effects (font (size 1.27 1.27)) hide)
-    )
-    (property "Datasheet" "" (id 3) (at 200.66 124.46 0)
-      (effects (font (size 1.27 1.27)) hide)
-    )
-    (pin "1")
   )
   (symbol (lib_id "RevK:LMR16006+FB") (at 49.53 131.445 0) (unit 1)
@@
     (property "Reference" "D2" (id 0) (at 83.185 22.4282 0))
     (property "Value" "D" (id 1) (at 83.185 24.7396 0))
-    (property "Footprint" "Diode_SMD:D_1206_3216Metric" (id 2) (at 83.185 27.94 0)
+    (property "Footprint" "RevK:D_1206" (id 2) (at 83.185 27.94 0)
       (effects (font (size 1.27 1.27)) hide)
     )
@@
       (reference "#PWR016") (unit 1) (value "+3.3V") (footprint "")
     )
-    (path "/1a8ea755-9b15-40ee-9e6d-e6e4769aa2cc"
-      (reference "#PWR017") (unit 1) (value "GND") (footprint "")
-    )
-    (path "/4d3b3a19-358a-434b-b4e1-15f15982ced7"
-      (reference "#PWR018") (unit 1) (value "+3.3V") (footprint "")
-    )
-    (path "/67f2d378-00dc-42d5-9279-3741999fa56c"
-      (reference "#PWR019") (unit 1) (value "+3.3V") (footprint "")
-    )
     (path "/d11ded20-64d4-49f4-9ed1-1e95f6ee0a71"
       (reference "#PWR020") (unit 1) (value "+3.3V") (footprint "")
@@
     )
     (path "/bbc62690-b8fb-438a-8ee0-c77d65956f89"
-      (reference "D2") (unit 1) (value "D") (footprint "Diode_SMD:D_1206_3216Metric")
+      (reference "D2") (unit 1) (value "D") (footprint "RevK:D_1206")
     )
     (path "/00000000-0000-0000-0000-000060cf36bc"
@@
       (reference "J2") (unit 1) (value "DC") (footprint "RevK:Molex_MiniSPOX_H2RA")
     )
-    (path "/3831277e-1b7d-4fa1-a209-da364bd7b5c6"
-      (reference "J3") (unit 1) (value "TEMP") (footprint "RevK:Molex_MiniSPOX_H3RA")
-    )
     (path "/00000000-0000-0000-0000-0000610fe01a"
       (reference "L1") (unit 1) (value "6.8uH") (footprint "RevK:Hidden")
@@
     )
     (path "/5d13f617-161f-4c68-98ea-696d87f0a0be"
-      (reference "M1") (unit 1) (value "EPaper") (footprint "")
+      (reference "M1") (unit 1) (value "EPaper") (footprint "Connector_PinHeader_2.54mm:PinHeader_1x13_P2.54mm_Vertical")
     )
     (path "/6324f539-5157-429d-ad08-999e5f3ad633"
@@
       (reference "R9") (unit 1) (value "10k") (footprint "RevK:R_0603")
     )
-    (path "/40905c56-15f1-4710-87cf-81fb9e340012"
-      (reference "R10") (unit 1) (value "4k7") (footprint "RevK:R_0603")
-    )
     (path "/00000000-0000-0000-0000-000060cf9e4d"
       (reference "R11") (unit 1) (value "680R") (footprint "RevK:R_0603")
@@
     )
     (path "/56ebf3fa-08d8-426b-9033-7d5fb9a0cae1"
-      (reference "U4") (unit 1) (value "QR") (footprint "RevK:QR-ENVMON")
-    )
-  )
+      (reference "U4") (unit 1) (value "QR") (footprint "RevK:QR-GFX")
+    )
+  )

Commit message: Epaper PCB
Parts:
- added H1, H2, H3, H4: MountingHole, RevK:Hole-2.5mm, symbol Mechanical:MountingHole
- added J3: Conn_01x02, RevK:Molex_MiniSPOX_H2RA, symbol Connector_Generic:Conn_01x02
- renumbered R11 to R10, R12 to R11, R13 to R12
Connections:
- net TEMP is gone; now on net SCK: U3.18 (IO14)
- net +3V3: now also M1.2 (3V3)
- net GND: now also M1.3 (GND), J3.1 (Pin_1)
- net SDCS: now reaches M1.10 (SDCS)
- net SDCS: now also U3.15 (IO25)
- net RST: now reaches M1.11 (RST)
- net RST: now also U3.16 (IO26)
- net BUSY: now reaches M1.12 (BUSY)
- net BUSY: now also U3.17 (IO27)
- net ENA: now reaches M1.13 (ENA)
- net ENA: now also U3.20 (IO13)
- net SCK: now reaches M1.4 (SCK)
- net MISO: now reaches M1.5 (MISO)
- net MISO: now also U3.12 (IO32)
- net MOSI: now reaches M1.6 (MOSI)
- net MOSI: now also U3.34 (IO22)
- net CS: now reaches M1.7 (ECS)
- net CS: now also U3.29 (IO5)
- net D/C: now reaches M1.8 (D/C)
- net D/C: now also U3.35 (IO21)
- net SRCS: now reaches M1.9 (SRCS)
- net SRCS: now also U3.13 (IO33)
- net BUTTON: now reaches U3.26 (IO20)
- net BUTTON: now also J3.2 (Pin_2)
- no-connect marks 16 -> 14

Commit message: Both epaper boards
Parts:
- J3: footprint RevK:Molex_MiniSPOX_H2RA -> RevK:Molex_MiniSPOX_H3RA; symbol Connector_Generic:Conn_01x02 -> Connector_Generic:Conn_01x03
Connections:
- net BUTTON1: now reaches U3.24 (IO4)
- net BUTTON1: now also J3.2 (Pin_2)
- net BUTTON renamed BUTTON2
- net BUTTON2: now also J3.3 (Pin_3); no longer J3.2 (Pin_2)
- no-connect marks 14 -> 13
Changed lines of the file:
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@@
   (no_connect (at 195.58 50.8))
   (no_connect (at 195.58 40.64))
-  (no_connect (at 195.58 63.5))
   (wire (pts (xy 55.88 33.02) (xy 58.42 33.02))
     (stroke (width 0) (type default) (color 0 0 0 0))
@@
     )
   )
+  (global_label "BUTTON2" (shape bidirectional) (at 198.12 104.14 180) (fields_autoplaced)
+    (effects (font (size 1.27 1.27)) (justify right))
+    (property "Intersheet References" "${INTERSHEET_REFS}" (id 0) (at 187.3896 104.0606 0)
+      (effects (font (size 1.27 1.27)) (justify right) hide)
+    )
+  )
   (global_label "BOOT" (shape input) (at 195.58 58.42 180) (fields_autoplaced)
     (effects (font (size 1.27 1.27)) (justify right))
@@
     )
   )
-  (global_label "BUTTON" (shape bidirectional) (at 198.12 104.14 180) (fields_autoplaced)
-    (effects (font (size 1.27 1.27)) (justify right))
-    (property "Intersheet References" "${INTERSHEET_REFS}" (id 0) (at 188.5991 104.0606 0)
+  (global_label "BUTTON1" (shape bidirectional) (at 198.12 101.6 180) (fields_autoplaced)
+    (effects (font (size 1.27 1.27)) (justify right))
+    (property "Intersheet References" "${INTERSHEET_REFS}" (id 0) (at 187.3896 101.5206 0)
       (effects (font (size 1.27 1.27)) (justify right) hide)
     )
@@
     )
   )
+  (global_label "BUTTON2" (shape bidirectional) (at 226.06 60.96 0) (fields_autoplaced)
+    (effects (font (size 1.27 1.27)) (justify left))
+    (property "Intersheet References" "${INTERSHEET_REFS}" (id 0) (at 236.7904 61.0394 0)
+      (effects (font (size 1.27 1.27)) (justify left) hide)
+    )
+  )
   (global_label "SRCS" (shape output) (at 226.06 78.74 0) (fields_autoplaced)
     (effects (font (size 1.27 1.27)) (justify left))
@@
     )
   )
-  (global_label "BUTTON" (shape bidirectional) (at 226.06 60.96 0) (fields_autoplaced)
-    (effects (font (size 1.27 1.27)) (justify left))
-    (property "Intersheet References" "${INTERSHEET_REFS}" (id 0) (at 235.5809 61.0394 0)
-      (effects (font (size 1.27 1.27)) (justify left) hide)
+  (global_label "BUTTON1" (shape bidirectional) (at 195.58 63.5 180) (fields_autoplaced)
+    (effects (font (size 1.27 1.27)) (justify right))
+    (property "Intersheet References" "${INTERSHEET_REFS}" (id 0) (at 184.8496 63.5794 0)
+      (effects (font (size 1.27 1.27)) (justify right) hide)
     )
   )
@@
     (pin "1")
   )
-  (symbol (lib_id "power:GND") (at 198.12 101.6 270) (unit 1)
+  (symbol (lib_id "power:GND") (at 198.12 99.06 270) (unit 1)
     (in_bom yes) (on_board yes) (fields_autoplaced)
-    (property "Reference" "#PWR019" (id 0) (at 191.77 101.6 0)
-      (effects (font (size 1.27 1.27)) hide)
-    )
-    (property "Value" "GND" (id 1) (at 194.9451 102.0338 90)
-      (effects (font (size 1.27 1.27)) (justify right))
-    )
-    (property "Footprint" "" (id 2) (at 198.12 101.6 0)
-      (effects (font (size 1.27 1.27)) hide)
-    )
-    (property "Datasheet" "" (id 3) (at 198.12 101.6 0)
+    (property "Reference" "#PWR019" (id 0) (at 191.77 99.06 0)
+      (effects (font (size 1.27 1.27)) hide)
+    )
+    (property "Value" "GND" (id 1) (at 194.9451 99.4938 90)
+      (effects (font (size 1.27 1.27)) (justify right))
+    )
+    (property "Footprint" "" (id 2) (at 198.12 99.06 0)
+      (effects (font (size 1.27 1.27)) hide)
+    )
+    (property "Datasheet" "" (id 3) (at 198.12 99.06 0)
       (effects (font (size 1.27 1.27)) hide)
     )
@@
     (pin "2")
   )
-  (symbol (lib_id "Connector_Generic:Conn_01x02") (at 203.2 101.6 0) (unit 1)
+  (symbol (lib_id "Connector_Generic:Conn_01x03") (at 203.2 101.6 0) (unit 1)
     (in_bom yes) (on_board yes) (fields_autoplaced)
     (property "Reference" "J3" (id 0) (at 205.232 102.0353 0)
@@
       (effects (font (size 1.27 1.27)) (justify left))
     )
-    (property "Footprint" "RevK:Molex_MiniSPOX_H2RA" (id 2) (at 203.2 101.6 0)
+    (property "Footprint" "RevK:Molex_MiniSPOX_H3RA" (id 2) (at 203.2 101.6 0)
       (effects (font (size 1.27 1.27)) hide)
     )
@@
     (pin "1")
     (pin "2")
+    (pin "3")
   )
   (symbol (lib_id "power:+3.3V") (at 226.06 38.1 270) (unit 1)
@@
     )
     (path "/ca6f103f-48cc-446d-9d86-158c35366e6f"
-      (reference "J3") (unit 1) (value "Conn_01x02") (footprint "RevK:Molex_MiniSPOX_H2RA")
+      (reference "J3") (unit 1) (value "Conn_01x02") (footprint "RevK:Molex_MiniSPOX_H3RA")
     )
     (path "/00000000-0000-0000-0000-0000610fe01a"

Commit message: Shelly as well for low power
Parts:
- added J2: Shelly, RevK:Shelly, symbol RevK:Shelly
- renumbered J2 to J3, J3 to J4
Connections:
- net +3V3: now also J2.3 (3V3)
- net BOOT: now also J2.2 (0)
- net GND: now also J2.1 (GND)
- net I: now also J2.5 (Tx)
- net O: now also J2.4 (Rx)
