File: PCB/EPD/EPD.kicad_sch (KiCad schematic)
At the start: 69 parts, among them J1 Conn_01x26, J2 Shelly, J3 USB-PROG, J4 BTN2, J6 BTN2, J7 USB-C-Socket-V, J8 PWR, P1 +, P10 2, P11 2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

Commit message: Caps, etc.
Changed lines of the file:
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@@
   (junction (at 161.29 109.855) (diameter 0) (color 0 0 0 0)
   )
+  (junction (at 262.89 84.455) (diameter 0) (color 0 0 0 0)
+  )
   (junction (at 187.96 88.265) (diameter 0) (color 0 0 0 0)
   )
@@
   (junction (at 161.29 102.235) (diameter 0) (color 0 0 0 0)
   )
-  (junction (at 262.89 84.455) (diameter 0) (color 0 0 0 0)
-  )
   (junction (at 253.365 147.955) (diameter 0) (color 0 0 0 0)
   )
@@
     )
   )
-  (symbol (lib_id "power:+3.3V") (at 60.96 24.765 0) (unit 1)
-    (in_bom yes) (on_board yes) (dnp no) (fields_autoplaced)
-    (property "Reference" "#PWR08" (at 60.96 28.575 0)
-      (effects (font (size 1.27 1.27)) hide)
+  (symbol (lib_id "Diode:1N5819") (at 266.7 84.455 180) (unit 1)
+    (in_bom yes) (on_board yes) (dnp no)
+    (property "Reference" "D6" (at 263.525 83.185 0)
+      (effects (font (size 1.27 1.27)))
     )
-    (property "Value" "+3.3V" (at 60.96 21.1892 0)
+    (property "Value" "MBR0530" (at 260.35 85.725 0)
       (effects (font (size 1.27 1.27)))
     )
-    (property "Footprint" "" (at 60.96 24.765 0)
+    (property "Footprint" "RevK:D_SOD-123" (at 266.7 80.01 0)
       (effects (font (size 1.27 1.27)) hide)
     )
-    (property "Datasheet" "" (at 60.96 24.765 0)
+    (property "Datasheet" "" (at 266.7 84.455 0)
+      (effects (font (size 1.27 1.27)) hide)
+    )
+    (property "LCSC Part #" "C5204746" (at 266.7 84.455 0)
       (effects (font (size 1.27 1.27)) hide)
     )
     (pin "1")
+    (pin "2")
     (instances
-      (project "USBA"
-        (path "/2d210a96-f81f-42a9-8bf4-1b43c11086f3"
-          (reference "#PWR08") (unit 1)
-        )
-      )
       (project "EPD"
         (path "/46c350bb-7de4-4e81-aafd-4af55e37aab0"
-          (reference "#PWR04") (unit 1)
+          (reference "D6") (unit 1)
         )
       )
     )
   )
-  (symbol (lib_id "Diode:1N5819") (at 266.7 84.455 180) (unit 1)
-    (in_bom yes) (on_board yes) (dnp no)
-    (property "Reference" "D6" (at 267.97 81.915 0)
-      (effects (font (size 1.27 1.27)))
+  (symbol (lib_id "power:+3.3V") (at 60.96 24.765 0) (unit 1)
+    (in_bom yes) (on_board yes) (dnp no) (fields_autoplaced)
+    (property "Reference" "#PWR08" (at 60.96 28.575 0)
+      (effects (font (size 1.27 1.27)) hide)
     )
-    (property "Value" "MBR0530" (at 271.145 80.01 0)
+    (property "Value" "+3.3V" (at 60.96 21.1892 0)
       (effects (font (size 1.27 1.27)))
     )
-    (property "Footprint" "RevK:D_SOD-123" (at 266.7 80.01 0)
-      (effects (font (size 1.27 1.27)) hide)
-    )
-    (property "Datasheet" "" (at 266.7 84.455 0)
+    (property "Footprint" "" (at 60.96 24.765 0)
       (effects (font (size 1.27 1.27)) hide)
     )
-    (property "LCSC Part #" "C5204746" (at 266.7 84.455 0)
+    (property "Datasheet" "" (at 60.96 24.765 0)
       (effects (font (size 1.27 1.27)) hide)
     )
     (pin "1")
-    (pin "2")
     (instances
+      (project "USBA"
+        (path "/2d210a96-f81f-42a9-8bf4-1b43c11086f3"
+          (reference "#PWR08") (unit 1)
+        )
+      )
       (project "EPD"
         (path "/46c350bb-7de4-4e81-aafd-4af55e37aab0"
-          (reference "D6") (unit 1)
+          (reference "#PWR04") (unit 1)
         )
       )
