File: PCB/EPD/EPD.kicad_sch (KiCad schematic)
At the start: 69 parts, among them J1 Conn_01x26, J2 Shelly, J3 USB-PROG, J4 BTN2, J6 BTN2, J7 USB-C-Socket-V, J8 PWR, P1 +, P10 2, P11 2, P12 2, P2 -, P3 2, P4 2, P5 2, P6 2, P7 +, P8 -, P9 2, Q1 BSS138, U2 ESP32-S3-MINI-1, U3 MD8942

Commit message: j
Parts:
- C8: value 10uF 50V -> 10uF 35V; LCSC Part # C1591 -> C194427
Changed lines of the file:
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@@
       (effects (font (size 1.27 1.27)) (justify left))
     )
-    (property "Value" "10uF 50V" (at 191.77 34.29 0)
+    (property "Value" "10uF 35V" (at 191.77 34.29 0)
       (effects (font (size 1.27 1.27)) (justify left))
     )
@@
       (effects (font (size 1.27 1.27)) hide)
     )
-    (property "LCSC Part #" "C1591" (at 185.42 34.29 0)
+    (property "LCSC Part #" "C194427" (at 185.42 34.29 0)
       (effects (font (size 1.27 1.27)) hide)
     )

Commit message: PCB Update
Parts:
- C8: LCSC Part # C194427 -> (none); MPN (none) -> C194427
- C9: LCSC Part # C1691 -> (none); MPN (none) -> C1691
- D1, D2, D3, D6: LCSC Part # C5204746 -> (none); MPN (none) -> C5204746
- D4: renamed from D1; LCSC Part # C5349953 -> (none); MPN (none) -> C5349953
- D5, D7: LCSC Part # C5137770 -> (none); MPN (none) -> C5137770
- J1: LCSC Part # C2856831 -> (none); MPN (none) -> C2856831
- J7: LCSC Part # C709357 -> (none); MPN (none) -> C709357
- Q1: JLCPCB Rotation Offset 180 -> (none); LCSC Part # C2938375 -> (none); MPN (none) -> C2938375
- U3: LCSC Part # C2684786 -> (none); MPN (none) -> C2684786
- U4: renamed from U2; LCSC Part # C3013941 -> (none); MPN (none) -> C3013941
- renumbered C3 to C1, C3 to C11, C3 to C12, C3 to C13, C3 to C14, C3 to C15, C3 to C16, C3 to C17, C3 to C18, C7 to C19, C1 to C2, C7 to C21, C3 to C4, C2 to C5, C3 to C6, C3 to C7, R1 to R2, R1 to R3, R2 to R4, R3 to R5, R12 to R6, R12 to R7, R1 to R8
