File: PCB/EPD75/EPD75.kicad_sch (KiCad schematic)
At the start: 132 parts, among them J1 Conn_01x26, J10 TF_PUSH, J2 Shelly, J3 USB-PROG, J4 BTN1, J5 USB-C-Socket-V, J6 BTN2, J7 USB-C-Socket-V, J8 PWR, J9 PWR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

Commit message: SD card
Parts:
- removed C5: 100nF, RevK:C_0402, symbol Device:C
- J4, J6, J8, J9: symbol Connector_Generic:Conn_01x02 -> Connector_Generic:Conn_01x04; now in the parts list
- R1: value 0.22R -> 0R47
Connections:
- net SPWR is gone; now on net +3.3V: J10.4 (VDD)
- net GND: now also J4.3 (Pin_3), J4.4 (Pin_4), J6.3 (Pin_3), J6.4 (Pin_4), J8.3 (Pin_3), J8.4 (Pin_4), J9.3 (Pin_3), J9.4 (Pin_4)
- net RELAY: now also U2.12 (GPIO8); no longer U2.28 (GPIO33)
- net RGB: now also U2.6 (GPIO2); no longer U2.29 (GPIO34)
- net SDCD: now also U2.11 (GPIO7)
- net SDMISO: now also U2.10 (GPIO6)
- net SDMOSI: now also U2.8 (GPIO4)
- net SDSCK: now also U2.9 (GPIO5)
- net SDSS: now also U2.7 (GPIO3)
- no-connect marks 30 -> 25
Other:
- moved on the sheet: C3, J2, J3, R1, U2

Commit message: BOM fix
Parts:
- J4, J6, J8, J9: now left out of the parts list
Changed lines of the file:
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@@
   )
   (symbol (lib_id "Connector_Generic:Conn_01x04") (at 278.765 28.575 0) (mirror x) (unit 1)
-    (in_bom yes) (on_board yes) (dnp no)
+    (in_bom no) (on_board yes) (dnp no)
     (property "Reference" "J6" (at 280.797 28.5171 0)
       (effects (font (size 1.27 1.27)) (justify left))
@@
   )
   (symbol (lib_id "Connector_Generic:Conn_01x04") (at 99.06 133.985 0) (unit 1)
-    (in_bom yes) (on_board yes) (dnp no)
+    (in_bom no) (on_board yes) (dnp no)
     (property "Reference" "J9" (at 101.092 134.0429 0)
       (effects (font (size 1.27 1.27)) (justify left))
@@
   )
   (symbol (lib_id "Connector_Generic:Conn_01x04") (at 231.14 63.5 0) (mirror x) (unit 1)
-    (in_bom yes) (on_board yes) (dnp no)
+    (in_bom no) (on_board yes) (dnp no)
     (property "Reference" "J8" (at 233.172 63.4421 0)
       (effects (font (size 1.27 1.27)) (justify left))
@@
   )
   (symbol (lib_id "Connector_Generic:Conn_01x04") (at 278.765 48.895 0) (mirror x) (unit 1)
-    (in_bom yes) (on_board yes) (dnp no)
+    (in_bom no) (on_board yes) (dnp no)
     (property "Reference" "J4" (at 280.797 48.8371 0)
       (effects (font (size 1.27 1.27)) (justify left))

Commit message: R
Parts:
- R1: value 0R47 -> 0.47R
Changed lines of the file:
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@@
       (effects (font (size 1.27 1.27)))
     )
-    (property "Value" "0R47" (at 183.515 157.48 90)
+    (property "Value" "0.47R" (at 183.515 157.48 90)
       (effects (font (size 1.27 1.27)))
     )

Commit message: j
Parts:
- C8: value 10uF 50V -> 10uF 35V; LCSC Part # C1591 -> C194427
- R9: LCSC Part # (none) -> C138062
Changed lines of the file:
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@@
       (effects (font (size 1.27 1.27)) hide)
     )
-    (property "Part No" "" (at 190.5 41.275 0)
-      (effects (font (size 1.27 1.27)) hide)
-    )
-    (property "Note" "" (at 190.5 41.275 0)
+    (property "LCSC Part #" "C138062" (at 190.5 41.275 0)
       (effects (font (size 1.27 1.27)) hide)
     )
@@
       (effects (font (size 1.27 1.27)) (justify left))
     )
-    (property "Value" "10uF 50V" (at 196.85 35.56 0)
+    (property "Value" "10uF 35V" (at 196.85 35.56 0)
       (effects (font (size 1.27 1.27)) (justify left))
     )
@@
       (effects (font (size 1.27 1.27)) hide)
     )
-    (property "LCSC Part #" "C1591" (at 190.5 35.56 0)
-      (effects (font (size 1.27 1.27)) hide)
-    )
+    (property "LCSC Part #" "C194427" (at 190.5 35.56 0)
+      (effects (font (size 1.27 1.27)) hide)
+    )

Commit message: New programming header
Parts:
- removed J2: Shelly, RevK:Shelly, symbol RevK:Shelly
- removed J3: USB-PROG, RevK:USB-PROG, symbol RevK:USB-PROG
- added J11: Reset, RevK:AA-Pad, symbol Connector_Generic:Conn_01x02
- added J12: TC2030-USB-NL-DS, RevK:Tag-Connect_TC2030-IDC-NL_2x03_P1.27mm_Vertical, symbol RevK:TC2030-USB-NL
Connections:
- net D+: now also J12.4 (D+)
- net D-: now also J12.3 (D-)
- net GND: now also J11.1 (Pin_1), J12.5 (GND), J12.6 (GND)
- net VBUS: now also J12.1 (VBUS), J12.2 (VBUS)
- net at U2.25 (GPIO21): now also J11.2 (Pin_2)
- no-connect marks 25 -> 27

Commit message: New connectors
Parts:
- removed J4: BTN1, RevK:PTSM-HH-2-RA-SMD, symbol Connector_Generic:Conn_01x04
- removed J6: BTN2, RevK:PTSM-HH-2-RA-SMD, symbol Connector_Generic:Conn_01x04
- removed J8, J9: PWR, RevK:PTSM-HH-2-RA-SMD, symbol Connector_Generic:Conn_01x04
- removed P41: -, RevK:SolderPad, symbol RevK:SolderPad
- removed P45: +, RevK:SolderPad, symbol RevK:SolderPad
- added J2, J8: PWR, RevK:WAGO-2060-452-998-404, symbol Connector_Generic:Conn_01x02
- added J3: RELAY, RevK:WAGO-2060-452-998-404, symbol Connector_Generic:Conn_01x02
- added J4: BTN1, RevK:WAGO-2060-452-998-404, symbol Connector_Generic:Conn_01x02
- added J6: BTN2, RevK:WAGO-2060-452-998-404, symbol Connector_Generic:Conn_01x02
- J11: now left out of the parts list
Connections:
- net GND: now also J2.1 (Pin_1), J4.1 (Pin_1), J6.1 (Pin_1), J8.1 (Pin_1)
- net PWR: now also J2.2 (Pin_2), J8.2 (Pin_2)
- net at D20.2, D34.2, D7.2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: now also J4.2 (Pin_2)
- net at D13.2, D27.2, D4.2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: now also J6.2 (Pin_2)
- net at P41.1 (P), U8.4: now also J3.2 (Pin_2)
- net at P45.1 (P), U8.3: now also J3.1 (Pin_1)

Commit message: Major tidy
Signed-off-by: RevK <github@e.gg>
Parts:
- removed D13, D20, D4, D7: ~, RevK:DFN1006-2L, symbol RevK:ES05D1MC10
- removed J2: PWR, RevK:WAGO-2060-452-998-404, symbol Connector_Generic:Conn_01x02
- removed P41, P45: O, RevK:SolderPad, symbol RevK:SolderPad
- removed P41, P42 (x2): -, RevK:SolderPad, symbol RevK:SolderPad
- removed P43: GND, RevK:SolderPad, symbol RevK:SolderPad
- removed P43 (x2): 2, RevK:SolderPad, symbol RevK:SolderPad
- removed P44 (x2): 1, RevK:SolderPad, symbol RevK:SolderPad
- removed P44: D+, RevK:SolderPad, symbol RevK:SolderPad
- removed P45, P46 (x2): +, RevK:SolderPad, symbol RevK:SolderPad
- removed P45: D-, RevK:SolderPad, symbol RevK:SolderPad
- removed P46: 5V, RevK:SolderPad, symbol RevK:SolderPad

Commit message: Clean
Connections:
- net at J3.1 (Pin_1): now also U8.4; no longer U8.3
- net at J3.2 (Pin_2): now also U8.3; no longer U8.4
Changed lines of the file:
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@@
 	(symbol
 		(lib_id "Connector_Generic:Conn_01x02")
-		(at 99.06 131.445 0)
+		(at 99.06 133.985 0)
+		(mirror x)
 		(unit 1)
 		(exclude_from_sim no)
@@
 		(dnp no)
 		(property "Reference" "J3"
-			(at 99.06 139.3995 0)
+			(at 99.06 126.0305 0)
 			(effects
 				(font
@@
 		)
 		(property "Value" "RELAY"
-			(at 99.06 136.9752 0)
+			(at 99.06 128.4548 0)
 			(effects
 				(font
@@
 		)
 		(property "Footprint" "RevK:WAGO-2060-452-998-404"
-			(at 99.06 131.445 0)
+			(at 99.06 133.985 0)
 			(effects
 				(font
@@
 		)
 		(property "Datasheet" "~"
-			(at 99.06 131.445 0)
+			(at 99.06 133.985 0)
 			(effects
 				(font
@@
 		)
 		(property "Description" "Generic connector, single row, 01x02, script generated (kicad-library-utils/schlib/autogen/connector/)"
-			(at 99.06 131.445 0)
+			(at 99.06 133.985 0)
 			(effects
 				(font
@@
 		)
 		(property "LCSC Part #" "C2765055"
-			(at 99.06 131.445 0)
+			(at 99.06 133.985 0)
 			(effects
 				(font
