File: PCB/EPD75/EPD75.kicad_pcb (KiCad board)
At the start: 2 copper layers, 168 x 110 mm, 108 parts, among them J1 Conn_01x26, J10 TF_PUSH, J11 Reset, J12 TC2030-USB-NL-DS, J3 RELAY, J4 BTN1, J5 USB-C-Socket-V, J6 BTN2, J7 USB-C-Socket-V, J8 PWR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

Commit message: Clean up
Parts:
- moved R14 28.5 mm to (135.0, 144.5)
- moved U1 22.5 mm to (138.5, 141.5), turned to 0 degrees
- moved R2 12.5 mm to (137.5, 59.0), turned to 0 degrees
- moved JP2 10.5 mm to (137.5, 61.6), turned to 90 degrees
- moved C18 10.4 mm to (124.9, 60.0), turned to 90 degrees
- moved R1 9.70 mm to (137.5, 64.2), turned to 180 degrees
- moved D3 8.81 mm to (134.9, 60.0), turned to -90 degrees
- moved L1 7.67 mm to (127.7, 60.0), turned to 90 degrees
- moved D1 7.18 mm to (132.9, 60.0), turned to -90 degrees
- moved D2 6.44 mm to (130.9, 60.0), turned to -90 degrees
- moved D34 6.10 mm to (147.5, 126.0), turned to 180 degrees
- moved D27 5.88 mm to (147.5, 64.0), turned to 180 degrees
- moved R4 5.05 mm to (147.8, 106.0)
- moved R5 4.83 mm to (147.8, 94.0)
- moved Q1 4.64 mm to (133.9, 64.1), turned to 180 degrees
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Routing:
- net +3.3V: track 902.8 -> 877.2 mm
- net Net-(J3-Pin_2): track 14.0 -> 37.8 mm
- net Net-(J3-Pin_1): track 14.0 -> 32.8 mm
- net Net-(J6-Pin_2): track 173.4 -> 156.1 mm
- net Net-(J4-Pin_2): track 154.7 -> 169.1 mm
- net RELAY: track 108.1 -> 118.5 mm
- net Net-(J7-CC2): track 1.39 -> 6.77 mm, vias 0 -> 2
- net Net-(J7-CC1): track 1.63 -> 7.01 mm, vias 0 -> 2
- net Net-(J1-Pin_3): track 52.7 -> 57.5 mm
- net Net-(J1-Pin_2): track 41.6 -> 45.9 mm
- net Net-(D3-K): track 45.5 -> 48.5 mm
- net Net-(D2-A): track 41.3 -> 40.1 mm
- net GND: track 21.2 -> 20.6 mm, vias 28 -> 42
Other:
- board text added: "epd.revk.uk"
- board text removed: "Secret Squirrel Certified"
- board text removed: "www.me.uk"

Commit message: Clean
Parts:
- moved R14 18.3 mm to (152.5, 139.0)
- moved U1 17.5 mm to (156.0, 141.5), turned to -90 degrees
- moved C12 7.18 mm to (89.5, 64.9), turned to -90 degrees
- moved C10 2.77 mm to (29.2, 76.0)
- moved C19 2.77 mm to (24.2, 73.0)
- moved C8 2.77 mm to (26.7, 75.3)
- moved C9 2.77 mm to (31.7, 75.3)
- moved D6 2.77 mm to (24.2, 78.0)
- moved L2 2.77 mm to (29.2, 78.6)
- moved R10 2.77 mm to (31.1, 72.1)
- moved R11 2.77 mm to (27.4, 72.1)
- moved R9 2.77 mm to (29.2, 72.1)
- moved U3 2.77 mm to (29.2, 74.0)
- moved J11 1.50 mm to (27.5, 62.0)
Connections:
- U1 pad 3: Net-(J3-Pin_1) -> Net-(J3-Pin_2)
- U1 pad 4: Net-(J3-Pin_2) -> Net-(J3-Pin_1)
Routing:
- net RELAY: track 118.5 -> 149.3 mm
- net +3.3V: track 877.2 -> 847.4 mm, vias 7 -> 9
- net D+: track 171.1 -> 198.2 mm
- net D-: track 173.9 -> 196.4 mm
- net BUSY: track 78.7 -> 98.1 mm
- net RST: track 80.4 -> 99.5 mm
- net DC: track 82.1 -> 100.9 mm
- net MOSI: track 87.1 -> 105.6 mm
- net CLK: track 85.4 -> 104.0 mm
- net CS: track 83.8 -> 102.2 mm
- net Net-(J4-Pin_2): track 169.1 -> 185.6 mm
- net PWR: track 164.6 -> 180.5 mm
- net Net-(D35-O): track 104.7 -> 117.5 mm
- net VBUS: track 232.1 -> 244.7 mm
- net Net-(J6-Pin_2): track 156.1 -> 166.6 mm
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
Commit message: Clean up
Parts:
- added R15: 10K, RevK:R_0402, F.Cu at (37.1, 119.1)
- added R16: 10K, RevK:R_0402, F.Cu at (37.1, 121.3)
- added R17: 10K, RevK:R_0402, F.Cu at (37.1, 116.9)
- moved C1 1.00 mm to (108.0, 58.2)
- moved C11 1.00 mm to (100.0, 58.5)
- moved C12 1.00 mm to (90.5, 64.9)
- moved C14 1.00 mm to (105.9, 58.5)
- moved C15 1.00 mm to (104.1, 58.5)
- moved C3 1.00 mm to (105.0, 58.5)
- moved C4 1.00 mm to (103.2, 58.5)
- moved C7 1.00 mm to (102.3, 58.5)
- moved J1 1.00 mm to (100.0, 66.0)
Routing:
- net Net-(D10-I): track 36.0 -> 41.2 mm
- net +3.3V: track 847.4 -> 852.0 mm
- net SDMISO: track 12.2 -> 13.9 mm
- net SDSCK: track 15.6 -> 17.0 mm
- net SDMOSI: track 16.6 -> 18.0 mm
- net DC: track 100.9 -> 101.9 mm
- net CS: track 102.2 -> 103.2 mm
- net Net-(J1-Pin_2): track 45.9 -> 44.9 mm
- net Net-(D2-A): track 40.1 -> 39.1 mm
- net Net-(J1-Pin_8): track 15.9 -> 16.9 mm
- net Net-(D3-K): track 48.6 -> 47.6 mm
- net CLK: track 104.0 -> 105.0 mm
- net RST: track 99.5 -> 100.5 mm
- net MOSI: track 105.6 -> 106.6 mm
- net BUSY: track 98.1 -> 99.1 mm
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Other:
- outline, holes or cut-outs redrawn
- board text added: "Board designed by RevK www.me.uk"
- board text added: "Line up the connector strip before fixing panel to board"
- board text added: "One USB at a time"
- board text added: "QR"
- board text added: "Use good quality adhesive such as 3M VHB tape"
- board text added: "®"

Commit message: Resistors
Parts:
- added R18: 10K, RevK:R_0402, F.Cu at (37.1, 119.1)
- added R19: 10K, RevK:R_0402, F.Cu at (37.1, 116.9)
- added R20: 10K, RevK:R_0402, F.Cu at (37.1, 115.8)
- moved R17 6.60 mm to (37.1, 123.5)
- moved R15 3.30 mm to (37.1, 122.4)
Connections:
- J10 pad 1: unconnected-(J10-DAT2-Pad1) -> Net-(J10-DAT2)
- J10 pad 8: unconnected-(J10-DAT1-Pad8) -> Net-(J10-DAT1)
- R15 pad 2: SDSCK -> SDSS
- R17 pad 2: SDMISO -> Net-(J10-DAT2)
Routing:
- net SDSS: track 18.8 -> 20.2 mm
- net Net-(J10-DAT2): track 0.00 -> 1.40 mm
- net Net-(J10-DAT1): track 0.00 -> 1.40 mm
- net +3.3V: track 852.0 -> 853.1 mm

Commit message: Tidy
Parts:
- added R21: 10K, RevK:R_0402, F.Cu at (37.1, 114.7)
Routing:
- net SDCD: track 11.1 -> 12.5 mm
- net +3.3V: track 853.1 -> 854.2 mm
Other:
- board text added: "No, not waterproof!"
