File: PCB/EPD75/EPD75.kicad_pcb (KiCad board)
At the start: 2 copper layers, 168 x 110 mm, 115 parts, among them J1 Conn_01x26, J10 TF_PUSH, J11 Reset, J12 TC2030-USB-NL-DS, J3 RELAY, J4 BTN1, J5 USB-C-Socket-V, J6 BTN2, J7 USB-C-Socket-V, J8 PWR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

Commit message: Silk screen
Other:
- board text added: "I could say something wise here, but once this is stuck down, it will never see the light of day ever again, so why bother."
- board text added: "Line up the connector strip before fixing panel to board Seriously, once stuck with 3M tape you are buggered!"
- board text added: "Secret Squirrel"
- board text added: "So, what can you do with this? Well, an interactive doorbell. Or a sign in a pub or restaurant. Or one your fridge to say bin day!"
- board text added: "This bit here means I can programme it with a TC2030 USB lead."
- board text added: "Use good quality adhesive such as 3M VHB tape 25mm x 50mm"
- board text removed: "Line up the connector strip before fixing panel to board"
- board text removed: "Use good quality adhesive such as 3M VHB tape"

Commit message: SS
Other:
- board text added: "So, what can you do with this? Well, an interactive doorbell. Or a sign in a pub or restaurant. Or on your fridge to say bin day!"
- board text removed: "So, what can you do with this? Well, an interactive doorbell. Or a sign in a pub or restaurant. Or one your fridge to say bin day!"

Commit message: NFC
Parts:
- moved J12 13.7 mm to (92.8, 139.2)
Routing:
- net D+: track 198.1 -> 224.8 mm, vias 2 -> 0
- net D-: track 196.4 -> 214.1 mm
- net Net-(J4-Pin_2): track 186.4 -> 199.6 mm
- net Net-(J1-Pin_2): track 44.9 -> 57.6 mm
- net VBUS: track 244.7 -> 257.1 mm
- net RELAY: track 149.3 -> 157.4 mm
- net Net-(J1-Pin_3): track 56.9 -> 59.4 mm
- net Net-(D3-K): track 47.6 -> 45.4 mm
- net +3.3V: track 854.2 -> 853.5 mm
- net Net-(D2-A): track 39.1 -> 38.5 mm
- net GND: vias 37 -> 45
Other:
- board text added: "Self adhesive pad for button-fix actually this side not on the front, like it says"
