File: PCB/EPD154/Epaper154.kicad_pcb (KiCad board)
At the start: 2 copper layers, 43.2 x 43.2 mm, 35 parts, among them J1 USB-C, J2 Shelly, J3 DC, J4 Conn_01x02, M1 EPaper, U1 LMR16006+FB, U2 FT231XQ, U3 ESP32-PICO-MINI-02, U4 QR

Commit message: QR
Parts:
- removed U4: QR, RevK:QR-GFX
- moved H1 39.7 mm to (169.5, 103.2), turned to -90 degrees
- moved H4 38.8 mm to (131.4, 103.2), turned to -90 degrees
- moved H2 37.5 mm to (169.5, 65.1), turned to -90 degrees
- moved H3 36.5 mm to (131.4, 65.1), turned to -90 degrees
- moved M1 33.0 mm to (131.4, 68.9), turned to 0 degrees
- moved D3 31.9 mm to (169.0, 70.8), turned to 180 degrees
- moved R11 30.6 mm to (169.0, 72.7), turned to 180 degrees
- moved R10 29.7 mm to (169.0, 74.0), turned to 180 degrees
- moved R12 29.0 mm to (169.0, 75.2), turned to 180 degrees
- moved R1 28.8 mm to (169.8, 78.0), turned to 90 degrees
- moved R2 27.1 mm to (168.5, 78.0), turned to -90 degrees
- moved L1 25.8 mm to (168.0, 86.3), turned to -90 degrees
- moved U1 25.4 mm to (168.0, 82.4), turned to -90 degrees
- moved C1 25.3 mm to (167.7, 80.3), turned to 0 degrees
- moved J1 23.2 mm to (150.4, 99.4), turned to 0 degrees
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Other:
- outline, holes or cut-outs redrawn
