File: PCB/EPD154/Epaper154.kicad_sch (KiCad schematic)
At the start: 35 parts, among them J1 USB-C, J2 Shelly, J3 DC, J4 Conn_01x02, M1 EPaper, U1 LMR16006+FB, U2 FT231XQ, U3 ESP32-PICO-MINI-02, U4 QR

Commit message: QR
Parts:
- removed U4: QR, RevK:QR-GFX, symbol RevK:QR
