File: PCB/EPDBat/EPDBat.kicad_sch (KiCad schematic)
At the start: 52 parts, among them J1 Conn_01x26, J3 JST-PH-SM3-TB, J4 Conn_01x02, J5 TC2030-USB-NL-DS, J7 USB-C-Socket-V, Q1 BSS138, Q1 C179347, Q4 CJ2301, U1 TP4054, U2 ESP32-S3-MINI-1, U2 ME6211C33M5G-N

Commit message: PCB Update
Parts:
- D1, D2, D3, D5: renamed from D4; LCSC Part  C5204746 -> (none); MPN (none) -> C5204746
- D4: renamed from D1; LCSC Part # C5349953 -> (none); MPN (none) -> C5349953
- D6: LCSC Part # C5137770 -> (none); MPN (none) -> C5137770
- J1: LCSC Part # C2856831 -> (none); MPN (none) -> C2856831
- J10: renamed from J3; footprint Connector_JST:JST_PH_S2B-PH-SM4-TB_1x02-1MP_P2.00mm_Horizontal -> RevK:JST_PH_S2B-PH-SM4-TB_1x02-1MP_P2.00mm_Horizontal; LCSC Part # C295747 -> (none); MPN (none) -> C295747
- J7: LCSC Part # C709357 -> (none); MPN (none) -> C709357
- Q1: JLCPCB Rotation Offset 180 -> (none); LCSC Part # C2938375 -> (none); MPN (none) -> C2938375
- Q2: renamed from Q4; JLCPCB Rotation Offset 180 -> (none); LCSC Part # C5224170 -> (none); MPN (none) -> C5224170
- Q3: renamed from Q1; LCSC Part # C179347 -> (none); MPN (none) -> C179347
- U1: JLCPCB Rotation Offset 180 -> (none); LCSC Part # C668215 -> (none); MPN (none) -> C668215
- U2: footprint Package_TO_SOT_SMD:SOT-23-5 -> RevK:SOT-23-5-90; JLCPCB Rotation Offset -90 -> (none); LCSC Part # C82942 -> (none); MPN (none) -> C82942
- U4: renamed from U2; LCSC Part # C3013941 -> (none); MPN (none) -> C3013941
- renumbered C3 to C1, C3 to C11, C3 to C12, C3 to C13, C3 to C14, C3 to C15, C3 to C16, C3 to C17, C3 to C18, C12 to C19, C1 to C2, C3 to C4, C2 to C5, C3 to C6, C3 to C7, R14 to R12, R15 to R13, R1 to R14, R12 to R16, R13 to R17, R1 to R2, R1 to R3, R2 to R4, R3 to R5, R1 to R8
